File: PCB/BurgerDisk-THT-Angled/BurgerDisk-THT-AngledDB19.kicad_pcb (KiCad board)
At the start: 2 copper layers, 93.7 x 86.9 mm, 18 parts, among them J1 Daisy port in, J2 MicroSD module, J3 UART, J4 Daisy port out, U1 PC817

Commit message: Update doc
Parts:
- moved G*** 65.8 mm to (143.0, 101.9)
- moved J2 14.0 mm to (144.2, 121.7)
Routing:
- net SCK: track 20.8 -> 40.0 mm
- net 5V_burgerDisk: track 79.8 -> 94.0 mm
- net MISO: track 20.9 -> 25.2 mm
- net CS: track 17.6 -> 21.9 mm
- net MOSI: track 20.4 -> 24.4 mm
- net GND: vias 33 -> 34
Other:
- board text added: "+/GND"
- board text added: "DB19-F"
- board text added: "TX/RX"
